Commit message: Address review of spot_description CHAMP changes

File: spot_description/urdf/spot.urdf.xacro (robot description, xacro)
@@ -5,6 +5,7 @@
   <!-- Parameters -->
   <xacro:arg name="arm" default="false" />
-  <xacro:arg name="tf_prefix" default="" />
+  <xacro:arg name="gazebo" default="false" />
+  <xacro:arg name="tf_prefix" default="false" />
   <!-- Load Spot -->
-  <xacro:load_spot arm="$(arg arm)" tf_prefix="$(arg tf_prefix)" />
+  <xacro:load_spot arm="$(arg arm)" gazebo="$(arg gazebo)" tf_prefix="$(arg tf_prefix)" />
 </robot>

File: spot_description/urdf/spot_leg.urdf.xacro (robot description, xacro)
@@ -1,24 +1,24 @@
 <?xml version="1.0"?>
 <robot xmlns:xacro="http://ros.org/wiki/xacro">
-    <xacro:macro name="spot_leg" params="leg_name tf_prefix " >
+    <xacro:macro name="spot_leg" params="leg_name tf_prefix ">
         <xacro:if value="${leg_name == 'front_left'}">
-            <xacro:property name="base_to_hip_xyz"            value="${base_to_hip_x} ${base_to_hip_y} 0" />
-            <xacro:property name="hip_to_upper_leg_xyz"       value="0 ${hip_to_upper_leg_y} 0" />
-            <xacro:property name="leg_side"                   value="left" />
+            <xacro:property name="base_to_hip_xyz" value="${base_to_hip_x} ${base_to_hip_y} 0" />
+            <xacro:property name="hip_to_upper_leg_xyz" value="0 ${hip_to_upper_leg_y} 0" />
+            <xacro:property name="leg_side" value="left" />
         </xacro:if>
         <xacro:if value="${leg_name == 'front_right'}">
-            <xacro:property name="base_to_hip_xyz"            value="${base_to_hip_x} -${base_to_hip_y} 0" />
-            <xacro:property name="hip_to_upper_leg_xyz"       value="0 -${hip_to_upper_leg_y} 0" />
-            <xacro:property name="leg_side"                   value="right" />
+            <xacro:property name="base_to_hip_xyz" value="${base_to_hip_x} -${base_to_hip_y} 0" />
+            <xacro:property name="hip_to_upper_leg_xyz" value="0 -${hip_to_upper_leg_y} 0" />
+            <xacro:property name="leg_side" value="right" />
         </xacro:if>
         <xacro:if value="${leg_name == 'rear_left'}">
-            <xacro:property name="base_to_hip_xyz"            value="-${base_to_hip_x} ${base_to_hip_y} 0" />
-            <xacro:property name="hip_to_upper_leg_xyz"       value="0 ${hip_to_upper_leg_y} 0" />
-            <xacro:property name="leg_side"                   value="left" />
+            <xacro:property name="base_to_hip_xyz" value="-${base_to_hip_x} ${base_to_hip_y} 0" />
+            <xacro:property name="hip_to_upper_leg_xyz" value="0 ${hip_to_upper_leg_y} 0" />
+            <xacro:property name="leg_side" value="left" />
         </xacro:if>
         <xacro:if value="${leg_name == 'rear_right'}">
-            <xacro:property name="base_to_hip_xyz"            value="-${base_to_hip_x} -${base_to_hip_y} 0" />
-            <xacro:property name="hip_to_upper_leg_xyz"       value="0 -${hip_to_upper_leg_y} 0" />
-            <xacro:property name="leg_side"                   value="right" />
+            <xacro:property name="base_to_hip_xyz" value="-${base_to_hip_x} -${base_to_hip_y} 0" />
+            <xacro:property name="hip_to_upper_leg_xyz" value="0 -${hip_to_upper_leg_y} 0" />
+            <xacro:property name="leg_side" value="right" />
         </xacro:if>
         <link name="${tf_prefix}${leg_name}_hip">
@@ -30,12 +30,11 @@
             <collision>
                 <geometry>
-                    <mesh filename="package://spot_description/meshes/base/collision/${leg_name}_hip_collision.obj" />
+                    <!-- Spot's hips' visual and collision geometry are identical. -->
+                    <mesh filename="package://spot_description/meshes/base/visual/${leg_name}_hip.obj" />
                 </geometry>
             </collision>
             <inertial>
                 <mass value="${hip_mass}"/>
-                <inertia ixx="${(1/12) * hip_mass * (hip_width * hip_width + hip_height * hip_height)}" ixy="0.0" ixz="0.0"
-                            iyy="${(1/12) * hip_mass * (hip_length * hip_length + hip_height * hip_height)}" iyz="0.0"
-                            izz="${(1/12) * hip_mass * (hip_length * hip_length + hip_width * hip_width)}" />
+                <inertia ixx="${(1/12) * hip_mass * (hip_width * hip_width + hip_height * hip_height)}" ixy="0.0" ixz="0.0" iyy="${(1/12) * hip_mass * (hip_length * hip_length + hip_height * hip_height)}" iyz="0.0" izz="${(1/12) * hip_mass * (hip_length * hip_length + hip_width * hip_width)}" />
             </inertial>
         </link>
@@ -61,7 +60,5 @@
                 <origin xyz="0 0 -0.14" rpy="0 0 0" />
                 <mass value="${upper_leg_mass}"/>
-                <inertia ixx="${(1/12) * upper_leg_mass * (upper_leg_width * upper_leg_width + upper_leg_height * upper_leg_height)}" ixy="0.0" ixz="0.0"
-                            iyy="${(1/12) * upper_leg_mass * (upper_leg_length * upper_leg_length + upper_leg_height * upper_leg_height)}" iyz="0.0"
-                            izz="${(1/12) * upper_leg_mass * (upper_leg_length * upper_leg_length + upper_leg_width * upper_leg_width)}" />
+                <inertia ixx="${(1/12) * upper_leg_mass * (upper_leg_width * upper_leg_width + upper_leg_height * upper_leg_height)}" ixy="0.0" ixz="0.0" iyy="${(1/12) * upper_leg_mass * (upper_leg_length * upper_leg_length + upper_leg_height * upper_leg_height)}" iyz="0.0" izz="${(1/12) * upper_leg_mass * (upper_leg_length * upper_leg_length + upper_leg_width * upper_leg_width)}" />
             </inertial>
         </link>
@@ -87,7 +84,5 @@
                 <origin xyz="0 0 -0.16" rpy="0 0 0" />
                 <mass value="${lower_leg_mass}"/>
-                <inertia ixx="${(1/12) * lower_leg_mass * (lower_leg_width * lower_leg_width + lower_leg_height * lower_leg_height)}" ixy="0.0" ixz="0.0"
-                            iyy="${(1/12) * lower_leg_mass * (lower_leg_length * lower_leg_length + lower_leg_height * lower_leg_height)}" iyz="0.0"
-                            izz="${(1/12) * lower_leg_mass * (lower_leg_length * lower_leg_length + lower_leg_width * lower_leg_width)}" />
+                <inertia ixx="${(1/12) * lower_leg_mass * (lower_leg_width * lower_leg_width + lower_leg_height * lower_leg_height)}" ixy="0.0" ixz="0.0" iyy="${(1/12) * lower_leg_mass * (lower_leg_length * lower_leg_length + lower_leg_height * lower_leg_height)}" iyz="0.0" izz="${(1/12) * lower_leg_mass * (lower_leg_length * lower_leg_length + lower_leg_width * lower_leg_width)}" />
             </inertial>
         </link>

File: spot_description/urdf/spot_macro.xacro (robot description, xacro)
@@ -59,8 +59,8 @@
         <!-- Macros for Spot's legs. -->
         <xacro:include filename="$(find spot_description)/urdf/spot_leg.urdf.xacro" />
-        <xacro:spot_leg leg_name="front_left"/>
-        <xacro:spot_leg leg_name="front_right"/>
-        <xacro:spot_leg leg_name="rear_left"/>
-        <xacro:spot_leg leg_name="rear_right"/>
+        <xacro:spot_leg leg_name="front_left" tf_prefix="${tf_prefix}"/>
+        <xacro:spot_leg leg_name="front_right" tf_prefix="${tf_prefix}"/>
+        <xacro:spot_leg leg_name="rear_left" tf_prefix="${tf_prefix}"/>
+        <xacro:spot_leg leg_name="rear_right" tf_prefix="${tf_prefix}"/>
         <!-- Standard accessories. -->
         <xacro:include filename="$(find spot_description)/urdf/accessories.urdf.xacro" />
@@ -70,5 +70,5 @@
         <xacro:if value="${arm}">
             <xacro:include filename="$(find spot_description)/urdf/spot_arm_macro.urdf" />
-            <xacro:load_arm tf_prefix="${tf_prefix}" />
+            <xacro:load_arm tf_prefix="${tf_prefix}"/>
         </xacro:if>
         <!-- Include Gazebo control if necessary -->

File: spot_description/urdf/standalone_arm.urdf.xacro (robot description, xacro)
@@ -1,4 +1,5 @@
 <?xml version="1.0"?>
-<robot name="standalone_arm" xmlns:xacro="http://www.ros.org/wiki/xacro">
+<robot name="standalone_arm"
+  xmlns:xacro="http://www.ros.org/wiki/xacro">
   <xacro:include filename="$(find spot_description)/urdf/spot_arm_macro.urdf" />
   <!-- Root link -->
@@ -7,5 +8,4 @@
   <xacro:arg name="tf_prefix" default="" />
   <!-- Load arm -->
-  <xacro:load_arm
-    tf_prefix="$(arg tf_prefix)" />
+  <xacro:load_arm tf_prefix="$(arg tf_prefix)" />
 </robot>
