Commit message: Convert URDF LIDAR control from env vars to xacro params

File: spot_description/urdf/accessories.urdf.xacro (robot description, xacro)
@@ -1,74 +1,76 @@
 <?xml version="1.0"?>
 <robot xmlns:xacro="http://www.ros.org/wiki/xacro">
-  <xacro:if value="$(optenv SPOT_PACK 0)">
-    <joint name="pack_mount_joint" type="fixed">
-      <parent link="base_link"/>
-      <child link="pack_mount"/>
-      <origin xyz="-0.019986 0 0.093662" rpy="0 0 0"/>
-    </joint>
-    <link name="pack_mount">
-      <visual>
-        <geometry>
-          <mesh filename="package://spot_description/meshes/base/visual/pack_top.obj"/>
-        </geometry>
-      </visual>
-      <visual>
-        <geometry>
-          <mesh filename="package://spot_description/meshes/base/visual/pack_body.obj"/>
-        </geometry>
-      </visual>
-      <collision>
-        <geometry>
-          <mesh filename="package://spot_description/meshes/base/visual/pack_body.obj"/>
-        </geometry>
-      </collision>
-    </link>
-  </xacro:if>
-  <xacro:if value="$(optenv SPOT_LIDAR_MOUNT 0)">
-    <joint name="lidar_mount_joint" type="fixed">
-      <parent link="pack_mount"/>
-      <child link="lidar_mount"/>
-      <origin xyz="0.015 0 0.149285" rpy="0 0 0"/>
-    </joint>
-    <link name="lidar_mount">
-      <visual>
-        <geometry>
-          <mesh filename="package://spot_description/meshes/base/visual/lidar_mount.obj"/>
-        </geometry>
-      </visual>
-      <collision>
-        <geometry>
-          <mesh filename="package://spot_description/meshes/base/collision/lidar_mount_collision.stl"/>
-        </geometry>
-      </collision>
-    </link>
-    <xacro:if value="$(optenv SPOT_VELODYNE 0)">
-      <!-- Use the Velodyne macro for the actual sensor -->
-      <xacro:include filename="$(find velodyne_description)/urdf/VLP-16.urdf.xacro" />
-      <xacro:VLP-16 parent="lidar_mount">
-        <origin xyz="$(optenv SPOT_VELODYNE_XYZ 0 0 0)" rpy="$(optenv SPOT_VELODYNE_RPY 0 0 0)" />
-      </xacro:VLP-16>
-      <!-- Add the protective cage -->
-      <link name="velodyne_cage">
+  <xacro:macro name="load_accessories" params="pack:=false lidar_mount:=false velodyne:=false velodyne_xyz:='0 0 0' velodyne_rpy:='0 0 0'">
+    <xacro:if value="${pack}">
+      <joint name="pack_mount_joint" type="fixed">
+        <parent link="base_link"/>
+        <child link="pack_mount"/>
+        <origin xyz="-0.019986 0 0.093662" rpy="0 0 0"/>
+      </joint>
+      <link name="pack_mount">
         <visual>
           <geometry>
-            <mesh filename="package://spot_description/meshes/base/collision/velodyne_cage.stl" scale="0.001 0.001 0.001" />
+            <mesh filename="package://spot_description/meshes/base/visual/pack_top.obj"/>
           </geometry>
-          <origin xyz="0 0 0" rpy="0 0 0" />
-          <material name="black" />
+        </visual>
+        <visual>
+          <geometry>
+            <mesh filename="package://spot_description/meshes/base/visual/pack_body.obj"/>
+          </geometry>
         </visual>
         <collision>
           <geometry>
-            <mesh filename="package://spot_description/meshes/base/collision/velodyne_cage.stl" scale="0.001 0.001 0.001" />
+            <mesh filename="package://spot_description/meshes/base/visual/pack_body.obj"/>
           </geometry>
-          <origin xyz="0 0 0" rpy="0 0 0" />
         </collision>
       </link>
-      <joint name="velodyne_cage_joint" type="fixed">
-        <parent link="lidar_mount" />
-        <child link="velodyne_cage" />
-        <origin xyz="$(optenv SPOT_VELODYNE_XYZ 0 0 0)" rpy="$(optenv SPOT_VELODYNE_RPY 0 0 0)" />
+    </xacro:if>
+    <xacro:if value="${lidar_mount}">
+      <joint name="lidar_mount_joint" type="fixed">
+        <parent link="pack_mount"/>
+        <child link="lidar_mount"/>
+        <origin xyz="0.015 0 0.149285" rpy="0 0 0"/>
       </joint>
+      <link name="lidar_mount">
+        <visual>
+          <geometry>
+            <mesh filename="package://spot_description/meshes/base/visual/lidar_mount.obj"/>
+          </geometry>
+        </visual>
+        <collision>
+          <geometry>
+            <mesh filename="package://spot_description/meshes/base/collision/lidar_mount_collision.stl"/>
+          </geometry>
+        </collision>
+      </link>
+      <xacro:if value="${velodyne}">
+        <!-- Use the Velodyne macro for the actual sensor -->
+        <xacro:include filename="$(find velodyne_description)/urdf/VLP-16.urdf.xacro" />
+        <xacro:VLP-16 parent="lidar_mount">
+          <origin xyz="${velodyne_xyz}" rpy="${velodyne_rpy}" />
+        </xacro:VLP-16>
+        <!-- Add the protective cage -->
+        <link name="velodyne_cage">
+          <visual>
+            <geometry>
+              <mesh filename="package://spot_description/meshes/base/collision/velodyne_cage.stl" scale="0.001 0.001 0.001" />
+            </geometry>
+            <origin xyz="0 0 0" rpy="0 0 0" />
+            <material name="black" />
+          </visual>
+          <collision>
+            <geometry>
+              <mesh filename="package://spot_description/meshes/base/collision/velodyne_cage.stl" scale="0.001 0.001 0.001" />
+            </geometry>
+            <origin xyz="0 0 0" rpy="0 0 0" />
+          </collision>
+        </link>
+        <joint name="velodyne_cage_joint" type="fixed">
+          <parent link="lidar_mount" />
+          <child link="velodyne_cage" />
+          <origin xyz="${velodyne_xyz}" rpy="${velodyne_rpy}" />
+        </joint>
+      </xacro:if>
     </xacro:if>
-  </xacro:if>
+  </xacro:macro>
 </robot>

File: spot_description/urdf/spot.urdf.xacro (robot description, xacro)
@@ -1,13 +1,12 @@
 <?xml version="1.0" ?>
-<robot name="spot" xmlns:xacro="http://www.ros.org/wiki/xacro">
+<robot name="spot"
+  xmlns:xacro="http://www.ros.org/wiki/xacro">
   <xacro:include filename="$(find spot_description)/urdf/spot_macro.xacro" />
   <!-- Parameters -->
   <xacro:arg name="arm" default="false" />
   <xacro:arg name="feet" default="false" />
+  <xacro:arg name="lidar" default="false" />
   <xacro:arg name="tf_prefix" default="" />
   <!-- Load Spot -->
-  <xacro:load_spot
-    arm="$(arg arm)"
-    feet="$(arg feet)"
-    tf_prefix="$(arg tf_prefix)" />
+  <xacro:load_spot arm="$(arg arm)" feet="$(arg feet)" lidar="$(arg lidar)" tf_prefix="$(arg tf_prefix)" />
 </robot>
