Commit message: Convert URDF LIDAR control from env vars to xacro params

File: spot_description/urdf/spot_macro.xacro (robot description, xacro)
@@ -1,8 +1,6 @@
 <?xml version="1.0"?>
-<robot name="spot" xmlns:xacro="http://www.ros.org/wiki/xacro">
-    <xacro:macro name="load_spot" params="
-    arm:=false
-    feet:=false
-    tf_prefix">
+<robot name="spot"
+    xmlns:xacro="http://www.ros.org/wiki/xacro">
+    <xacro:macro name="load_spot" params="arm feet lidar tf_prefix">
         <link name="${tf_prefix}body">
             <visual>
@@ -13,6 +11,5 @@
             <collision>
                 <geometry>
-                    <mesh
-                        filename="package://spot_description/meshes/base/collision/body_collision.obj" />
+                    <mesh filename="package://spot_description/meshes/base/collision/body_collision.obj" />
                 </geometry>
             </collision>
@@ -20,9 +17,7 @@
         <link name="${tf_prefix}base_link">
             <inertial>
-                <origin rpy="0.0 0.0 0.0"
-                    xyz="0.006394396536052227 -9.812158532440662e-05 0.0009113792330026627" />
+                <origin rpy="0.0 0.0 0.0" xyz="0.006394396536052227 -9.812158532440662e-05 0.0009113792330026627" />
                 <mass value="32.86" />
-                <inertia ixx="0.13143999874591827" ixy="0.0" ixz="0.0" iyy="0.13143999874591827"
-                    iyz="0.0" izz="0.13143999874591827" />
+                <inertia ixx="0.13143999874591827" ixy="0.0" ixz="0.0" iyy="0.13143999874591827" iyz="0.0" izz="0.13143999874591827" />
             </inertial>
         </link>
@@ -59,14 +54,11 @@
             <visual>
                 <geometry>
-                    <mesh
-                        filename="package://spot_description/meshes/base/visual/front_left_hip.obj" />
-                </geometry>
-            </visual>
-            <inertial>
-                <origin rpy="-0.716521349312305 0.02956473059648479 0.03655230014702582"
-                    xyz="-0.005374345928430557 0.012841847725212574 9.875232353806496e-05" />
+                    <mesh filename="package://spot_description/meshes/base/visual/front_left_hip.obj" />
+                </geometry>
+            </visual>
+            <inertial>
+                <origin rpy="-0.716521349312305 0.02956473059648479 0.03655230014702582" xyz="-0.005374345928430557 0.012841847725212574 9.875232353806496e-05" />
                 <mass value="1.68" />
-                <inertia ixx="0.0021147398873455382" ixy="0.0" ixz="0.0" iyy="0.0018129577956607131"
-                    iyz="0.0" izz="0.002265435737304666" />
+                <inertia ixx="0.0021147398873455382" ixy="0.0" ixz="0.0" iyy="0.0018129577956607131" iyz="0.0" izz="0.002265435737304666" />
             </inertial>
         </link>
@@ -76,26 +68,21 @@
             <parent link="${tf_prefix}body" />
             <child link="${tf_prefix}front_left_hip" />
-            <limit effort="45" velocity="17.647" lower="-0.78539816339744827899"
-                upper="0.78539816339744827899" />
+            <limit effort="45" velocity="17.647" lower="-0.78539816339744827899" upper="0.78539816339744827899" />
         </joint>
         <link name="${tf_prefix}front_left_upper_leg">
             <visual>
                 <geometry>
-                    <mesh
-                        filename="package://spot_description/meshes/base/visual/front_left_upper_leg.obj" />
-                </geometry>
-            </visual>
-            <collision>
-                <geometry>
-                    <mesh
-                        filename="package://spot_description/meshes/base/collision/left_upper_leg_collision.obj" />
-                </geometry>
-            </collision>
-            <inertial>
-                <origin rpy="-0.26437828203369795 -0.04853174570753804 0.024046963096353124"
-                    xyz="0.005142373498529196 -0.0024323679972440004 -0.12100915610790253" />
+                    <mesh filename="package://spot_description/meshes/base/visual/front_left_upper_leg.obj" />
+                </geometry>
+            </visual>
+            <collision>
+                <geometry>
+                    <mesh filename="package://spot_description/meshes/base/collision/left_upper_leg_collision.obj" />
+                </geometry>
+            </collision>
+            <inertial>
+                <origin rpy="-0.26437828203369795 -0.04853174570753804 0.024046963096353124" xyz="0.005142373498529196 -0.0024323679972440004 -0.12100915610790253" />
                 <mass value="2.34" />
-                <inertia ixx="0.02755964961185679" ixy="0.0" ixz="0.0" iyy="0.027354914287651046"
-                    iyz="0.0" izz="0.002848145546743553" />
+                <inertia ixx="0.02755964961185679" ixy="0.0" ixz="0.0" iyy="0.027354914287651046" iyz="0.0" izz="0.002848145546743553" />
             </inertial>
         </link>
@@ -105,18 +92,15 @@
             <parent link="${tf_prefix}front_left_hip" />
             <child link="${tf_prefix}front_left_upper_leg" />
-            <limit effort="45" velocity="17.647" lower="-0.89884456477707963539"
-                upper="2.2951079663725435509" />
+            <limit effort="45" velocity="17.647" lower="-0.89884456477707963539" upper="2.2951079663725435509" />
         </joint>
         <link name="${tf_prefix}front_left_lower_leg">
             <visual>
                 <geometry>
-                    <mesh
-                        filename="package://spot_description/meshes/base/visual/front_left_lower_leg.obj" />
-                </geometry>
-            </visual>
-            <collision>
-                <geometry>
-                    <mesh
-                        filename="package://spot_description/meshes/base/collision/left_lower_leg_collision.obj" />
+                    <mesh filename="package://spot_description/meshes/base/visual/front_left_lower_leg.obj" />
+                </geometry>
+            </visual>
+            <collision>
+                <geometry>
+                    <mesh filename="package://spot_description/meshes/base/collision/left_lower_leg_collision.obj" />
                 </geometry>
             </collision>
@@ -128,9 +112,7 @@
             </collision>
             <inertial>
-                <origin rpy="-0.007266925694167092 -0.009591807116834161 0.00035255970529224356"
-                    xyz="0.00225794012658298 4.607596201822162e-05 -0.1800822913646698" />
+                <origin rpy="-0.007266925694167092 -0.009591807116834161 0.00035255970529224356" xyz="0.00225794012658298 4.607596201822162e-05 -0.1800822913646698" />
                 <mass value="0.35" />
-                <inertia ixx="0.003999022654901177" ixy="0.0" ixz="0.0" iyy="0.0040503157598010785"
-                    iyz="0.0" izz="0.0001493402097647426" />
+                <inertia ixx="0.003999022654901177" ixy="0.0" ixz="0.0" iyy="0.0040503157598010785" iyz="0.0" izz="0.0001493402097647426" />
             </inertial>
         </link>
@@ -145,14 +127,11 @@
             <visual>
                 <geometry>
-                    <mesh
-                        filename="package://spot_description/meshes/base/visual/front_right_hip.obj" />
-                </geometry>
-            </visual>
-            <inertial>
-                <origin rpy="0.7165213493123055 -0.02956473059648479 0.03655230014702582"
-                    xyz="-0.005374345928430557 -0.012841847725212574 -9.875232353806496e-05" />
+                    <mesh filename="package://spot_description/meshes/base/visual/front_right_hip.obj" />
+                </geometry>
+            </visual>
+            <inertial>
+                <origin rpy="0.7165213493123055 -0.02956473059648479 0.03655230014702582" xyz="-0.005374345928430557 -0.012841847725212574 -9.875232353806496e-05" />
                 <mass value="1.68" />
-                <inertia ixx="0.0021147398873455382" ixy="0.0" ixz="0.0" iyy="0.0018129577956607131"
-                    iyz="0.0" izz="0.002265435737304666" />
+                <inertia ixx="0.0021147398873455382" ixy="0.0" ixz="0.0" iyy="0.0018129577956607131" iyz="0.0" izz="0.002265435737304666" />
             </inertial>
         </link>
@@ -162,26 +141,21 @@
             <parent link="${tf_prefix}body" />
             <child link="${tf_prefix}front_right_hip" />
-            <limit effort="45" velocity="17.647" lower="-0.78539816339744827899"
-                upper="0.78539816339744827899" />
+            <limit effort="45" velocity="17.647" lower="-0.78539816339744827899" upper="0.78539816339744827899" />
         </joint>
         <link name="${tf_prefix}front_right_upper_leg">
             <visual>
                 <geometry>
-                    <mesh
-                        filename="package://spot_description/meshes/base/visual/front_right_upper_leg.obj" />
-                </geometry>
-            </visual>
-            <collision>
-                <geometry>
-                    <mesh
-                        filename="package://spot_description/meshes/base/collision/right_upper_leg_collision.obj" />
-                </geometry>
-            </collision>
-            <inertial>
-                <origin rpy="0.2643905306958363 -0.04853174688302708 -0.024046943559834943"
-                    xyz="0.005142373498529196 0.0024323677644133568 -0.12100915610790253" />
+                    <mesh filename="package://spot_description/meshes/base/visual/front_right_upper_leg.obj" />
+                </geometry>
+            </visual>
+            <collision>
+                <geometry>
+                    <mesh filename="package://spot_description/meshes/base/collision/right_upper_leg_collision.obj" />
+                </geometry>
+            </collision>
+            <inertial>
+                <origin rpy="0.2643905306958363 -0.04853174688302708 -0.024046943559834943" xyz="0.005142373498529196 0.0024323677644133568 -0.12100915610790253" />
                 <mass value="2.34" />
-                <inertia ixx="0.02755964678927691" ixy="0.0" ixz="0.0" iyy="0.02735491706466737"
-                    iyz="0.0" izz="0.0028481453594764797" />
+                <inertia ixx="0.02755964678927691" ixy="0.0" ixz="0.0" iyy="0.02735491706466737" iyz="0.0" izz="0.0028481453594764797" />
             </inertial>
         </link>
@@ -191,18 +165,15 @@
             <parent link="${tf_prefix}front_right_hip" />
             <child link="${tf_prefix}front_right_upper_leg" />
-            <limit effort="45" velocity="17.647" lower="-0.89884456477707963539"
-                upper="2.2951079663725435509" />
+            <limit effort="45" velocity="17.647" lower="-0.89884456477707963539" upper="2.2951079663725435509" />
         </joint>
         <link name="${tf_prefix}front_right_lower_leg">
             <visual>
                 <geometry>
-                    <mesh
-                        filename="package://spot_description/meshes/base/visual/front_right_lower_leg.obj" />
-                </geometry>
-            </visual>
-            <collision>
-                <geometry>
-                    <mesh
-                        filename="package://spot_description/meshes/base/collision/right_lower_leg_collision.obj" />
+                    <mesh filename="package://spot_description/meshes/base/visual/front_right_lower_leg.obj" />
+                </geometry>
+            </visual>
+            <collision>
+                <geometry>
+                    <mesh filename="package://spot_description/meshes/base/collision/right_lower_leg_collision.obj" />
                 </geometry>
             </collision>
@@ -214,9 +185,7 @@
             </collision>
             <inertial>
-                <origin rpy="-0.007266925694167092 -0.009591807116834161 0.00035255970529224356"
-                    xyz="0.00225794012658298 4.607596201822162e-05 -0.1800822913646698" />
+                <origin rpy="-0.007266925694167092 -0.009591807116834161 0.00035255970529224356" xyz="0.00225794012658298 4.607596201822162e-05 -0.1800822913646698" />
                 <mass value="0.35" />
-                <inertia ixx="0.003999022654901177" ixy="0.0" ixz="0.0" iyy="0.0040503157598010785"
-                    iyz="0.0" izz="0.0001493402097647426" />
+                <inertia ixx="0.003999022654901177" ixy="0.0" ixz="0.0" iyy="0.0040503157598010785" iyz="0.0" izz="0.0001493402097647426" />
             </inertial>
         </link>
@@ -231,14 +200,11 @@
             <visual>
                 <geometry>
-                    <mesh
-                        filename="package://spot_description/meshes/base/visual/rear_left_hip.obj" />
-                </geometry>
-            </visual>
-            <inertial>
-                <origin rpy="0.7165213493123055 -0.02956473059648479 0.03655230014702582"
-                    xyz="-0.005374345928430557 -0.012841847725212574 -9.875232353806496e-05" />
+                    <mesh filename="package://spot_description/meshes/base/visual/rear_left_hip.obj" />
+                </geometry>
+            </visual>
+            <inertial>
+                <origin rpy="0.7165213493123055 -0.02956473059648479 0.03655230014702582" xyz="-0.005374345928430557 -0.012841847725212574 -9.875232353806496e-05" />
                 <mass value="1.68" />
-                <inertia ixx="0.0021147398873455382" ixy="0.0" ixz="0.0" iyy="0.0018129577956607131"
-                    iyz="0.0" izz="0.002265435737304666" />
+                <inertia ixx="0.0021147398873455382" ixy="0.0" ixz="0.0" iyy="0.0018129577956607131" iyz="0.0" izz="0.002265435737304666" />
             </inertial>
         </link>
@@ -248,26 +214,21 @@
             <parent link="${tf_prefix}body" />
             <child link="${tf_prefix}rear_left_hip" />
-            <limit effort="45" velocity="17.647" lower="-0.78539816339744827899"
-                upper="0.78539816339744827899" />
+            <limit effort="45" velocity="17.647" lower="-0.78539816339744827899" upper="0.78539816339744827899" />
         </joint>
         <link name="${tf_prefix}rear_left_upper_leg">
             <visual>
                 <geometry>
-                    <mesh
-                        filename="package://spot_description/meshes/base/visual/rear_left_upper_leg.obj" />
-                </geometry>
-            </visual>
-            <collision>
-                <geometry>
-                    <mesh
-                        filename="package://spot_description/meshes/base/collision/left_upper_leg_collision.obj" />
-                </geometry>
-            </collision>
-            <inertial>
-                <origin rpy="-0.26437828203369795 -0.04853174570753804 0.024046963096353124"
-                    xyz="0.005142373498529196 -0.0024323679972440004 -0.12100915610790253" />
+                    <mesh filename="package://spot_description/meshes/base/visual/rear_left_upper_leg.obj" />
+                </geometry>
+            </visual>
+            <collision>
+                <geometry>
+                    <mesh filename="package://spot_description/meshes/base/collision/left_upper_leg_collision.obj" />
+                </geometry>
+            </collision>
+            <inertial>
+                <origin rpy="-0.26437828203369795 -0.04853174570753804 0.024046963096353124" xyz="0.005142373498529196 -0.0024323679972440004 -0.12100915610790253" />
                 <mass value="2.34" />
-                <inertia ixx="0.02755964961185679" ixy="0.0" ixz="0.0" iyy="0.027354914287651046"
-                    iyz="0.0" izz="0.002848145546743553" />
+                <inertia ixx="0.02755964961185679" ixy="0.0" ixz="0.0" iyy="0.027354914287651046" iyz="0.0" izz="0.002848145546743553" />
             </inertial>
         </link>
@@ -277,18 +238,15 @@
             <parent link="${tf_prefix}rear_left_hip" />
             <child link="${tf_prefix}rear_left_upper_leg" />
-            <limit effort="45" velocity="17.647" lower="-0.89884456477707963539"
-                upper="2.2951079663725435509" />
+            <limit effort="45" velocity="17.647" lower="-0.89884456477707963539" upper="2.2951079663725435509" />
         </joint>
         <link name="${tf_prefix}rear_left_lower_leg">
             <visual>
                 <geometry>
-                    <mesh
-                        filename="package://spot_description/meshes/base/visual/rear_left_lower_leg.obj" />
-                </geometry>
-            </visual>
-            <collision>
-                <geometry>
-                    <mesh
-                        filename="package://spot_description/meshes/base/collision/left_lower_leg_collision.obj" />
+                    <mesh filename="package://spot_description/meshes/base/visual/rear_left_lower_leg.obj" />
+                </geometry>
+            </visual>
+            <collision>
+                <geometry>
+                    <mesh filename="package://spot_description/meshes/base/collision/left_lower_leg_collision.obj" />
                 </geometry>
             </collision>
@@ -300,9 +258,7 @@
             </collision>
             <inertial>
-                <origin rpy="-0.007266925694167092 -0.009591807116834161 0.00035255970529224356"
-                    xyz="0.00225794012658298 4.607596201822162e-05 -0.1800822913646698" />
+                <origin rpy="-0.007266925694167092 -0.009591807116834161 0.00035255970529224356" xyz="0.00225794012658298 4.607596201822162e-05 -0.1800822913646698" />
                 <mass value="0.35" />
-                <inertia ixx="0.003999022654901177" ixy="0.0" ixz="0.0" iyy="0.0040503157598010785"
-                    iyz="0.0" izz="0.0001493402097647426" />
+                <inertia ixx="0.003999022654901177" ixy="0.0" ixz="0.0" iyy="0.0040503157598010785" iyz="0.0" izz="0.0001493402097647426" />
             </inertial>
         </link>
@@ -317,14 +273,11 @@
             <visual>
                 <geometry>
-                    <mesh
-                        filename="package://spot_description/meshes/base/visual/rear_right_hip.obj" />
-                </geometry>
-            </visual>
-            <inertial>
-                <origin rpy="0.7165213493123055 -0.02956473059648479 0.03655230014702582"
-                    xyz="-0.005374345928430557 -0.012841847725212574 -9.875232353806496e-05" />
+                    <mesh filename="package://spot_description/meshes/base/visual/rear_right_hip.obj" />
+                </geometry>
+            </visual>
+            <inertial>
+                <origin rpy="0.7165213493123055 -0.02956473059648479 0.03655230014702582" xyz="-0.005374345928430557 -0.012841847725212574 -9.875232353806496e-05" />
                 <mass value="1.68" />
-                <inertia ixx="0.0021147398873455382" ixy="0.0" ixz="0.0" iyy="0.0018129577956607131"
-                    iyz="0.0" izz="0.002265435737304666" />
+                <inertia ixx="0.0021147398873455382" ixy="0.0" ixz="0.0" iyy="0.0018129577956607131" iyz="0.0" izz="0.002265435737304666" />
             </inertial>
         </link>
@@ -334,26 +287,21 @@
             <parent link="${tf_prefix}body" />
             <child link="${tf_prefix}rear_right_hip" />
-            <limit effort="45" velocity="17.647" lower="-0.78539816339744827899"
-                upper="0.78539816339744827899" />
+            <limit effort="45" velocity="17.647" lower="-0.78539816339744827899" upper="0.78539816339744827899" />
         </joint>
         <link name="${tf_prefix}rear_right_upper_leg">
             <visual>
                 <geometry>
-                    <mesh
-                        filename="package://spot_description/meshes/base/visual/rear_right_upper_leg.obj" />
-                </geometry>
-            </visual>
-            <collision>
-                <geometry>
-                    <mesh
-                        filename="package://spot_description/meshes/base/collision/right_upper_leg_collision.obj" />
-                </geometry>
-            </collision>
-            <inertial>
-                <origin rpy="0.2643905306958363 -0.04853174688302708 -0.024046943559834943"
-                    xyz="0.005142373498529196 0.0024323677644133568 -0.12100915610790253" />
+                    <mesh filename="package://spot_description/meshes/base/visual/rear_right_upper_leg.obj" />
+                </geometry>
+            </visual>
+            <collision>
+                <geometry>
+                    <mesh filename="package://spot_description/meshes/base/collision/right_upper_leg_collision.obj" />
+                </geometry>
+            </collision>
+            <inertial>
+                <origin rpy="0.2643905306958363 -0.04853174688302708 -0.024046943559834943" xyz="0.005142373498529196 0.0024323677644133568 -0.12100915610790253" />
                 <mass value="2.34" />
-                <inertia ixx="0.02755964678927691" ixy="0.0" ixz="0.0" iyy="0.02735491706466737"
-                    iyz="0.0" izz="0.0028481453594764797" />
+                <inertia ixx="0.02755964678927691" ixy="0.0" ixz="0.0" iyy="0.02735491706466737" iyz="0.0" izz="0.0028481453594764797" />
             </inertial>
         </link>
@@ -363,18 +311,15 @@
             <parent link="${tf_prefix}rear_right_hip" />
             <child link="${tf_prefix}rear_right_upper_leg" />
-            <limit effort="45" velocity="17.647" lower="-0.89884456477707963539"
-                upper="2.2951079663725435509" />
+            <limit effort="45" velocity="17.647" lower="-0.89884456477707963539" upper="2.2951079663725435509" />
         </joint>
         <link name="${tf_prefix}rear_right_lower_leg">
             <visual>
                 <geometry>
-                    <mesh
-                        filename="package://spot_description/meshes/base/visual/rear_right_lower_leg.obj" />
-                </geometry>
-            </visual>
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