Commit message: WIP: Add local changes

File: spot_description/urdf/accessories.urdf.xacro (robot description, xacro)
@@ -2,31 +2,7 @@
 <robot xmlns:xacro="http://www.ros.org/wiki/xacro">
   <xacro:macro name="load_accessories" params="pack:=false lidar_mount:=false velodyne:=false velodyne_xyz:='0 0 0' velodyne_rpy:='0 0 0'">
-    <xacro:if value="${pack}">
-      <joint name="pack_mount_joint" type="fixed">
-        <parent link="base_link"/>
-        <child link="pack_mount"/>
-        <origin xyz="-0.019986 0 0.093662" rpy="0 0 0"/>
-      </joint>
-      <link name="pack_mount">
-        <visual>
-          <geometry>
-            <mesh filename="package://spot_description/meshes/base/visual/pack_top.obj"/>
-          </geometry>
-        </visual>
-        <visual>
-          <geometry>
-            <mesh filename="package://spot_description/meshes/base/visual/pack_body.obj"/>
-          </geometry>
-        </visual>
-        <collision>
-          <geometry>
-            <mesh filename="package://spot_description/meshes/base/visual/pack_body.obj"/>
-          </geometry>
-        </collision>
-      </link>
-    </xacro:if>
     <xacro:if value="${lidar_mount}">
       <joint name="lidar_mount_joint" type="fixed">
-        <parent link="pack_mount"/>
+        <parent link="base_link"/>
         <child link="lidar_mount"/>
         <origin xyz="0.015 0 0.149285" rpy="0 0 0"/>

File: spot_description/urdf/spot_macro.xacro (robot description, xacro)
@@ -344,10 +344,10 @@
         </joint>
         <!-- Include LIDAR if requested -->
-        <xacro:include filename="$(find spot_description)/urdf/accessories.urdf.xacro" />
-        <xacro:load_accessories pack="true" lidar_mount="true" velodyne="true" />
-        <!--  <xacro:if value="${lidar}">
+        <!--<xacro:include filename="$(find spot_description)/urdf/accessories.urdf.xacro" />
+        <xacro:load_accessories pack="true" lidar_mount="true" velodyne="true" />-->
+        <xacro:if value="${lidar}">
             <xacro:include filename="$(find spot_description)/urdf/accessories.urdf.xacro" />
-            <xacro:load_accessories pack="true" lidar_mount="true" velodyne="true" />
-        </xacro:if>-->
+            <xacro:load_accessories pack="false" lidar_mount="true" velodyne="true" />
+        </xacro:if>
         <!-- Optional custom includes -->
         <xacro:include filename="$(optenv SPOT_URDF_EXTRAS empty.urdf)" />

Commit message: Edit URDF constants and formatting

File: spot_description/urdf/accessories.urdf.xacro (robot description, xacro)
@@ -3,22 +3,22 @@
   <xacro:if value="$(optenv SPOT_PACK 0)">
     <joint name="pack_mount_joint" type="fixed">
-      <parent link="base_link"/>
-      <child link="pack_mount"/>
-      <origin xyz="-0.019986 0 0.093662" rpy="0 0 0"/>
+      <parent link="base_link" />
+      <child link="pack_mount" />
+      <origin xyz="-0.019986 0 0.093662" rpy="0 0 0" />
     </joint>
     <link name="pack_mount">
       <visual>
         <geometry>
-          <mesh filename="package://spot_description/meshes/base/visual/pack_top.obj"/>
+          <mesh filename="package://spot_description/meshes/base/visual/pack_top.obj" />
         </geometry>
       </visual>
       <visual>
         <geometry>
-          <mesh filename="package://spot_description/meshes/base/visual/pack_body.obj"/>
+          <mesh filename="package://spot_description/meshes/base/visual/pack_body.obj" />
         </geometry>
       </visual>
       <collision>
         <geometry>
-          <mesh filename="package://spot_description/meshes/base/visual/pack_body.obj"/>
+          <mesh filename="package://spot_description/meshes/base/visual/pack_body.obj" />
         </geometry>
       </collision>
@@ -27,17 +27,18 @@
   <xacro:if value="$(optenv SPOT_LIDAR_MOUNT 0)">
     <joint name="lidar_mount_joint" type="fixed">
-      <parent link="pack_mount"/>
-      <child link="lidar_mount"/>
-      <origin xyz="0.015 0 0.149285" rpy="0 0 0"/>
+      <parent link="pack_mount" />
+      <child link="lidar_mount" />
+      <origin xyz="0.015 0 0.149285" rpy="0 0 0" />
     </joint>
     <link name="lidar_mount">
       <visual>
         <geometry>
-          <mesh filename="package://spot_description/meshes/base/visual/lidar_mount.obj"/>
+          <mesh filename="package://spot_description/meshes/base/visual/lidar_mount.obj" />
         </geometry>
       </visual>
       <collision>
         <geometry>
-          <mesh filename="package://spot_description/meshes/base/collision/lidar_mount_collision.stl"/>
+          <mesh
+            filename="package://spot_description/meshes/base/collision/lidar_mount_collision.stl" />
         </geometry>
       </collision>
@@ -53,5 +54,6 @@
         <visual>
           <geometry>
-            <mesh filename="package://spot_description/meshes/base/collision/velodyne_cage.stl" scale="0.001 0.001 0.001" />
+            <mesh filename="package://spot_description/meshes/base/collision/velodyne_cage.stl"
+              scale="0.001 0.001 0.001" />
           </geometry>
           <origin xyz="0 0 0" rpy="0 0 0" />
@@ -60,5 +62,6 @@
         <collision>
           <geometry>
-            <mesh filename="package://spot_description/meshes/base/collision/velodyne_cage.stl" scale="0.001 0.001 0.001" />
+            <mesh filename="package://spot_description/meshes/base/collision/velodyne_cage.stl"
+              scale="0.001 0.001 0.001" />
           </geometry>
           <origin xyz="0 0 0" rpy="0 0 0" />
@@ -72,10 +75,11 @@
     </xacro:if>
   </xacro:if>
-  <xacro:if value="$(optenv CHAMP_GAZEBO 0)">
+  <xacro:if value="${gazebo}">
     <xacro:include filename="$(find spot_description)/urdf/constants.urdf.xacro" />
     <xacro:include filename="$(find hector_sensors_description)/urdf/hokuyo_utm30lx.urdf.xacro" />
     <xacro:include filename="$(find hector_sensors_description)/urdf/asus_camera.urdf.xacro" />
-    <xacro:hokuyo_utm30lx name="hokuyo" parent="base_link" ros_topic="scan" update_rate="30" ray_count="1040" min_angle="130" max_angle="-130">
-      <origin xyz="0.0 0.0 ${base_height / 2 + 0.04}" rpy="0 0 0"/>
+    <xacro:hokuyo_utm30lx name="hokuyo" parent="base_link" ros_topic="scan" update_rate="30"
+      ray_count="1040" min_angle="130" max_angle="-130">
+      <origin xyz="0.0 0.0 ${base_height / 2 + 0.04}" rpy="0 0 0" />
     </xacro:hokuyo_utm30lx>
     <gazebo reference="hokuyo_frame">
@@ -83,5 +87,5 @@
     </gazebo>
     <xacro:asus_camera parent="base_link" name="camera">
-      <origin xyz="${base_length / 2 - 0.05} 0.0 -${base_height / 2 + 0.01}" rpy="0 0 0"/>
+      <origin xyz="${base_length / 2 - 0.05} 0.0 -${base_height / 2 + 0.01}" rpy="0 0 0" />
     </xacro:asus_camera>
     <gazebo>
@@ -100,7 +104,7 @@
     <link name="imu_link">
       <inertial>
-        <mass value="0.001"/>
-        <origin xyz="0 0 0" rpy="0 0 0"/>
-        <inertia ixx="1e-09" ixy="0.0" ixz="0.0" iyy="1e-09" iyz="0.0" izz="1e-09"/>
+        <mass value="0.001" />
+        <origin xyz="0 0 0" rpy="0 0 0" />
+        <inertia ixx="1e-09" ixy="0.0" ixz="0.0" iyy="1e-09" iyz="0.0" izz="1e-09" />
       </inertial>
     </link>

File: spot_description/urdf/constants.urdf.xacro (robot description, xacro)
@@ -6,18 +6,24 @@
     <xacro:property name="upper_leg_to_lower_leg_x" value="0.025" />
     <xacro:property name="upper_leg_to_lower_leg_z" value="0.3205" />
-    <xacro:property name="lower_leg_to_foot_z" value="0.37" />
-    <xacro:property name="base_mass" value="16.0" />
-    <xacro:property name="base_length" value="0.86" />
-    <xacro:property name="base_width" value="0.21" />
-    <xacro:property name="base_height" value="0.17" />
-    <xacro:property name="hip_mass" value="2.0" />
+    <!-- Distance from foot to knee (meters) -->
+    <xacro:property name="lower_leg_to_foot_z" value="0.35" />
+    <!-- Values from the URDF provided by the Spot SDK -->
+    <!-- https://dev.bostondynamics.com/docs/concepts/joint_control/supplemental_data.html -->
+    <xacro:property name="base_mass" value="16.70765207" />
+    <xacro:property name="base_length" value="0.85" />
+    <xacro:property name="base_width" value="0.24" />
+    <xacro:property name="base_height" value="0.18" />
+    <!-- Mass per the URDF provided by the Spot SDK -->
+    <xacro:property name="hip_mass" value="1.13688339" />
     <xacro:property name="hip_length" value="0.13" />
     <xacro:property name="hip_width" value="0.09" />
     <xacro:property name="hip_height" value="0.09" />
-    <xacro:property name="upper_leg_mass" value="1.0" />
+    <!-- Mass per the URDF provided by the Spot SDK -->
+    <xacro:property name="upper_leg_mass" value="2.25620359" />
     <xacro:property name="upper_leg_length" value="0.076" />
     <xacro:property name="upper_leg_width" value="0.076" />
     <xacro:property name="upper_leg_height" value="0.425" />
-    <xacro:property name="lower_leg_mass" value="0.5" />
+    <!-- Mass per the URDF provided by the Spot SDK (Spot ROS 2 driver says 0.35 kg) -->
+    <xacro:property name="lower_leg_mass" value="0.33" />
     <xacro:property name="lower_leg_length" value="0.035" />
     <xacro:property name="lower_leg_width" value="0.045" />

File: spot_description/urdf/spot.urdf.xacro (robot description, xacro)
@@ -1,8 +1,8 @@
-<?xml version="1.0" ?>
+<?xml version="1.0"?>
 <robot name="spot"
   xmlns:xacro="http://www.ros.org/wiki/xacro">
   <xacro:include filename="$(find spot_description)/urdf/spot_macro.xacro" />
   <!-- Parameters -->
-  <xacro:arg name="arm" default="false" />
+  <xacro:arg name="arm" default="true" />
   <xacro:arg name="gazebo" default="false" />
   <xacro:arg name="tf_prefix" default="" />

File: spot_description/urdf/spot_leg.urdf.xacro (robot description, xacro)
@@ -1,5 +1,5 @@
 <?xml version="1.0"?>
 <robot xmlns:xacro="http://ros.org/wiki/xacro">
-    <xacro:macro name="spot_leg" params="leg_name tf_prefix ">
+    <xacro:macro name="spot_leg" params="leg_name tf_prefix gazebo">
         <xacro:if value="${leg_name == 'front_left'}">
             <xacro:property name="base_to_hip_xyz" value="${base_to_hip_x} ${base_to_hip_y} 0" />
@@ -25,5 +25,6 @@
             <visual>
                 <geometry>
-                    <mesh filename="package://spot_description/meshes/base/visual/${leg_name}_hip.obj" />
+                    <mesh
+                        filename="package://spot_description/meshes/base/visual/${leg_name}_hip.obj" />
                 </geometry>
             </visual>
@@ -31,10 +32,17 @@
                 <geometry>
                     <!-- Spot's hips' visual and collision geometry are identical. -->
-                    <mesh filename="package://spot_description/meshes/base/visual/${leg_name}_hip.obj" />
+                    <mesh
+                        filename="package://spot_description/meshes/base/visual/${leg_name}_hip.obj" />
                 </geometry>
             </collision>
             <inertial>
-                <mass value="${hip_mass}"/>
-                <inertia ixx="${(1/12) * hip_mass * (hip_width * hip_width + hip_height * hip_height)}" ixy="0.0" ixz="0.0" iyy="${(1/12) * hip_mass * (hip_length * hip_length + hip_height * hip_height)}" iyz="0.0" izz="${(1/12) * hip_mass * (hip_length * hip_length + hip_width * hip_width)}" />
+                <mass value="${hip_mass}" />
+                <inertia
+                    ixx="${(1/12) * hip_mass * (hip_width * hip_width + hip_height * hip_height)}"
+                    ixy="0.0"
+                    ixz="0.0"
+                    iyy="${(1/12) * hip_mass * (hip_length * hip_length + hip_height * hip_height)}"
+                    iyz="0.0"
+                    izz="${(1/12) * hip_mass * (hip_length * hip_length + hip_width * hip_width)}" />
             </inertial>
         </link>
@@ -44,21 +52,29 @@
             <parent link="${tf_prefix}body" />
             <child link="${tf_prefix}${leg_name}_hip" />
-            <limit effort="45" velocity="17.647" lower="-0.78539816339744827899" upper="0.78539816339744827899" />
+            <limit effort="45" velocity="17.647" lower="-0.78539816339744827899"
+                upper="0.78539816339744827899" />
         </joint>
         <link name="${tf_prefix}${leg_name}_upper_leg">
             <visual>
                 <geometry>
-                    <mesh filename="package://spot_description/meshes/base/visual/${leg_name}_upper_leg.obj" />
+                    <mesh
+                        filename="package://spot_description/meshes/base/visual/${leg_name}_upper_leg.obj" />
                 </geometry>
             </visual>
             <collision>
                 <geometry>
-                    <mesh filename="package://spot_description/meshes/base/collision/${leg_side}_upper_leg_collision.obj" />
+                    <mesh
+                        filename="package://spot_description/meshes/base/collision/${leg_side}_upper_leg_collision.obj" />
                 </geometry>
             </collision>
             <inertial>
                 <origin xyz="0 0 -0.14" rpy="0 0 0" />
-                <mass value="${upper_leg_mass}"/>
-                <inertia ixx="${(1/12) * upper_leg_mass * (upper_leg_width * upper_leg_width + upper_leg_height * upper_leg_height)}" ixy="0.0" ixz="0.0" iyy="${(1/12) * upper_leg_mass * (upper_leg_length * upper_leg_length + upper_leg_height * upper_leg_height)}" iyz="0.0" izz="${(1/12) * upper_leg_mass * (upper_leg_length * upper_leg_length + upper_leg_width * upper_leg_width)}" />
+                <mass value="${upper_leg_mass}" />
+                <inertia
+                    ixx="${(1/12) * upper_leg_mass * (upper_leg_width * upper_leg_width + upper_leg_height * upper_leg_height)}"
+                    ixy="0.0" ixz="0.0"
+                    iyy="${(1/12) * upper_leg_mass * (upper_leg_length * upper_leg_length + upper_leg_height * upper_leg_height)}"
+                    iyz="0.0"
+                    izz="${(1/12) * upper_leg_mass * (upper_leg_length * upper_leg_length + upper_leg_width * upper_leg_width)}" />
             </inertial>
         </link>
@@ -68,31 +84,41 @@
             <parent link="${tf_prefix}${leg_name}_hip" />
             <child link="${tf_prefix}${leg_name}_upper_leg" />
-            <limit effort="45" velocity="17.647" lower="-0.89884456477707963539" upper="2.2951079663725435509" />
+            <limit effort="45" velocity="17.647" lower="-0.89884456477707963539"
+                upper="2.2951079663725435509" />
         </joint>
         <link name="${tf_prefix}${leg_name}_lower_leg">
             <visual>
                 <geometry>
-                    <mesh filename="package://spot_description/meshes/base/visual/${leg_name}_lower_leg.obj" />
+                    <mesh
+                        filename="package://spot_description/meshes/base/visual/${leg_name}_lower_leg.obj" />
                 </geometry>
             </visual>
             <collision>
                 <geometry>
-                    <mesh filename="package://spot_description/meshes/base/collision/${leg_side}_lower_leg_collision.obj" />
+                    <mesh
+                        filename="package://spot_description/meshes/base/collision/${leg_side}_lower_leg_collision.obj" />
                 </geometry>
             </collision>
             <inertial>
                 <origin xyz="0 0 -0.16" rpy="0 0 0" />
-                <mass value="${lower_leg_mass}"/>
-                <inertia ixx="${(1/12) * lower_leg_mass * (lower_leg_width * lower_leg_width + lower_leg_height * lower_leg_height)}" ixy="0.0" ixz="0.0" iyy="${(1/12) * lower_leg_mass * (lower_leg_length * lower_leg_length + lower_leg_height * lower_leg_height)}" iyz="0.0" izz="${(1/12) * lower_leg_mass * (lower_leg_length * lower_leg_length + lower_leg_width * lower_leg_width)}" />
+                <mass value="${lower_leg_mass}" />
+                <inertia
+                    ixx="${(1/12) * lower_leg_mass * (lower_leg_width * lower_leg_width + lower_leg_height * lower_leg_height)}"
+                    ixy="0.0" ixz="0.0"
+                    iyy="${(1/12) * lower_leg_mass * (lower_leg_length * lower_leg_length + lower_leg_height * lower_leg_height)}"
+                    iyz="0.0"
+                    izz="${(1/12) * lower_leg_mass * (lower_leg_length * lower_leg_length + lower_leg_width * lower_leg_width)}" />
             </inertial>
         </link>
-        <gazebo reference="${tf_prefix}${leg_name}_lower_leg">
-            <kp>100000.0</kp>
-            <kd>1.0</kd>
-            <mu1>0.8</mu1>
-            <mu2>0.8</mu2>
-            <maxVel>0.0</maxVel>
-            <minDepth>0.001</minDepth>
-        </gazebo>
+        <xacro:if value="${gazebo}">
+            <gazebo reference="${tf_prefix}${leg_name}_lower_leg">
+                <kp>100000.0</kp>
+                <kd>1.0</kd>
+                <mu1>0.8</mu1>
+                <mu2>0.8</mu2>
+                <maxVel>0.0</maxVel>
+                <minDepth>0.001</minDepth>
+            </gazebo>
+        </xacro:if>
         <joint name="${tf_prefix}${leg_name}_knee" type="revolute">
             <origin xyz="${upper_leg_to_lower_leg_x} 0 -${upper_leg_to_lower_leg_z}" rpy="0 0 0" />

File: spot_description/urdf/spot_macro.xacro (robot description, xacro)
@@ -1,8 +1,6 @@
 <?xml version="1.0"?>
-<robot name="spot"
-    xmlns:xacro="http://www.ros.org/wiki/xacro">
+<robot name="spot" xmlns:xacro="http://www.ros.org/wiki/xacro">
     <xacro:include filename="$(find spot_description)/urdf/constants.urdf.xacro" />
-    <xacro:macro name="load_spot" params=" arm:=false gazebo:=false
-    tf_prefix">
+    <xacro:macro name="load_spot" params="arm:=false gazebo:=false tf_prefix">
         <link name="${tf_prefix}body">
             <visual>
@@ -13,17 +11,26 @@
             <collision>
                 <geometry>
-                    <mesh filename="package://spot_description/meshes/base/collision/body_collision.obj" />
+                    <mesh
+                        filename="package://spot_description/meshes/base/collision/body_collision.obj" />
                 </geometry>
             </collision>
             <inertial>
-                <mass value="${base_mass}"/>
-                <inertia ixx="${(1/12) * base_mass * (base_width * base_width + base_height * base_height)}" ixy="0.0" ixz="0.0" iyy="${(1/12) * base_mass * (base_length * base_length + base_height * base_height)}" iyz="0.0" izz="${(1/12) * base_mass * (base_length * base_length + base_width * base_width)}" />
+                <mass value="${base_mass}" />
+                <inertia
+                    ixx="${(1/12) * base_mass * (base_width * base_width + base_height * base_height)}"
+                    ixy="0.0"
+                    ixz="0.0"
+                    iyy="${(1/12) * base_mass * (base_length * base_length + base_height * base_height)}"
+                    iyz="0.0"
+                    izz="${(1/12) * base_mass * (base_length * base_length + base_width * base_width)}" />
             </inertial>
         </link>
         <link name="${tf_prefix}base_link">
             <inertial>
-                <origin rpy="0.0 0.0 0.0" xyz="0.006394396536052227 -9.812158532440662e-05 0.0009113792330026627" />
+                <origin rpy="0.0 0.0 0.0"
+                    xyz="0.006394396536052227 -9.812158532440662e-05 0.0009113792330026627" />
                 <mass value="32.86" />
-                <inertia ixx="0.13143999874591827" ixy="0.0" ixz="0.0" iyy="0.13143999874591827" iyz="0.0" izz="0.13143999874591827" />
+                <inertia ixx="0.13143999874591827" ixy="0.0" ixz="0.0" iyy="0.13143999874591827"
+                    iyz="0.0" izz="0.13143999874591827" />
             </inertial>
         </link>
@@ -59,8 +66,8 @@
         <!-- Macros for Spot's legs. -->
         <xacro:include filename="$(find spot_description)/urdf/spot_leg.urdf.xacro" />
-        <xacro:spot_leg leg_name="front_left" tf_prefix="${tf_prefix}"/>
-        <xacro:spot_leg leg_name="front_right" tf_prefix="${tf_prefix}"/>
-        <xacro:spot_leg leg_name="rear_left" tf_prefix="${tf_prefix}"/>
-        <xacro:spot_leg leg_name="rear_right" tf_prefix="${tf_prefix}"/>
+        <xacro:spot_leg leg_name="front_left" tf_prefix="${tf_prefix}" gazebo="${gazebo}" />
+        <xacro:spot_leg leg_name="front_right" tf_prefix="${tf_prefix}" gazebo="${gazebo}" />
+        <xacro:spot_leg leg_name="rear_left" tf_prefix="${tf_prefix}" gazebo="${gazebo}" />
+        <xacro:spot_leg leg_name="rear_right" tf_prefix="${tf_prefix}" gazebo="${gazebo}" />
         <!-- Standard accessories. -->
         <xacro:include filename="$(find spot_description)/urdf/accessories.urdf.xacro" />
@@ -70,5 +77,5 @@
         <xacro:if value="${arm}">
             <xacro:include filename="$(find spot_description)/urdf/spot_arm_macro.urdf" />
-            <xacro:load_arm tf_prefix="${tf_prefix}"/>
+            <xacro:load_arm tf_prefix="${tf_prefix}" />
         </xacro:if>
         <!-- Include Gazebo control if necessary -->
