Commit message: Commit current changes

File: spot_description/urdf/spot.urdf (robot description, URDF)
Before this commit: robot spot, 28 links, 27 joints
Links:
- removed link Falsearm_link_el0
- removed link Falsearm_link_el1
- removed link Falsearm_link_fngr
- removed link Falsearm_link_hr0
- removed link Falsearm_link_sh0
- removed link Falsearm_link_sh1
- removed link Falsearm_link_wr0
- removed link Falsearm_link_wr1
- removed link Falsebase_link
- removed link Falsebody
- removed link Falsefront_left_ee
- removed link Falsefront_left_hip
- removed link Falsefront_left_lower_leg
- removed link Falsefront_left_upper_leg
- removed link Falsefront_rail
- removed link Falsefront_right_ee
- removed link Falsefront_right_hip
- removed link Falsefront_right_lower_leg
- removed link Falsefront_right_upper_leg
- removed link Falserear_left_ee
- removed link Falserear_left_hip
- removed link Falserear_left_lower_leg
- removed link Falserear_left_upper_leg
- removed link Falserear_rail
- removed link Falserear_right_ee
- removed link Falserear_right_hip
- removed link Falserear_right_lower_leg
- removed link Falserear_right_upper_leg
- added link arm_link_el0, mass 0.725; collision mesh filename=package://spot_description/meshes/arm/collision/arm_link_el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; visual mesh filename=package://spot_description/meshes/arm/visual/arm_link_el0.o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
- added link arm_link_el1, mass 0.725; collision mesh filename=package://spot_description/meshes/arm/collision/arm_link_el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; collision mesh filename=package://spot_description/meshes/arm/collision/arm_link_el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
- added link arm_link_fngr, mass 0.2; collision mesh filename=package://spot_description/meshes/arm/collision/left_finger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; collision mesh filename=package://spot_description/meshes/arm/collision/left_hinge.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
- added link arm_link_hr0, mass 1e-06; collision mesh filename=package://spot_description/meshes/arm/collision/arm_link_hr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; visual mesh filename=package://spot_description/meshes/arm/visual/arm_link_hr0.o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
- added link arm_link_sh0, mass 2.3364000000000003; collision mesh filename=package://spot_description/meshes/arm/collision/arm_link_sh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; collision mesh filename=package://spot_description/meshes/arm/collision/arm_link_sh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
- added link arm_link_sh1, mass 0.2596; visual mesh filename=package://spot_description/meshes/arm/visual/arm_link_sh1.o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
- added link arm_link_wr0, mass 0.98; collision mesh filename=package://spot_description/meshes/arm/collision/arm_link_wr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; visual mesh filename=package://spot_description/meshes/arm/visual/arm_link_wr0.o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
- added link arm_link_wr1, mass 0.785; collision mesh filename=package://spot_description/meshes/arm/collision/arm_link_wr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; collision mesh filename=package://spot_description/meshes/arm/collision/front_jaw.o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
- added link base_link, mass 32.86
- added link body, mass 16.70765207; collision mesh filename=package://spot_description/meshes/base/collision/body_colli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; visual mesh filename=package://spot_description/meshes/base/visual/body.obj
- added link front_left_ee
- added link front_left_hip, mass 1.13688339; collision mesh filename=package://spot_description/meshes/base/visual/front_left_hi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; visual mesh filename=package://spot_description/meshes/base/visual/front_left_hi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
- added link front_left_lower_leg, mass 0.33; collision mesh filename=package://spot_description/meshes/base/collision/left_lower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; visual mesh filename=package://spot_description/meshes/base/visual/front_left_lo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
- added link front_left_upper_leg, mass 2.25620359; collision mesh filename=package://spot_description/meshes/base/collision/left_upper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; visual mesh filename=package://spot_description/meshes/base/visual/front_left_up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
- added link front_rail, mass 1.0e-6
- added link front_right_ee
- added link front_right_hip, mass 1.13688339; collision mesh filename=package://spot_description/meshes/base/visual/front_right_h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; visual mesh filename=package://spot_description/meshes/base/visual/front_right_h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
- added link front_right_lower_leg, mass 0.33; collision mesh filename=package://spot_description/meshes/base/collision/right_lowe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; visual mesh filename=package://spot_description/meshes/base/visual/front_right_l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
- added link front_right_upper_leg, mass 2.25620359; collision mesh filename=package://spot_description/meshes/base/collision/right_uppe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; visual mesh filename=package://spot_description/meshes/base/visual/front_right_u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
- added link rear_left_ee
- added link rear_left_hip, mass 1.13688339; collision mesh filename=package://spot_description/meshes/base/visual/rear_left_hip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; visual mesh filename=package://spot_description/meshes/base/visual/rear_left_hip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
- added link rear_left_lower_leg, mass 0.33; collision mesh filename=package://spot_description/meshes/base/collision/left_lower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; visual mesh filename=package://spot_description/meshes/base/visual/rear_left_low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
- added link rear_left_upper_leg, mass 2.25620359; collision mesh filename=package://spot_description/meshes/base/collision/left_upper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; visual mesh filename=package://spot_description/meshes/base/visual/rear_left_upp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
- added link rear_rail, mass 1.0e-6
- added link rear_right_ee
- added link rear_right_hip, mass 1.13688339; collision mesh filename=package://spot_description/meshes/base/visual/rear_right_hi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; visual mesh filename=package://spot_description/meshes/base/visual/rear_right_hi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
- added link rear_right_lower_leg, mass 0.33; collision mesh filename=package://spot_description/meshes/base/collision/right_lowe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; visual mesh filename=package://spot_description/meshes/base/visual/rear_right_lo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
- added link rear_right_upper_leg, mass 2.25620359; collision mesh filename=package://spot_description/meshes/base/collision/right_uppe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; visual mesh filename=package://spot_description/meshes/base/visual/rear_right_up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
Joints:
- removed joint Falsearm_el0
- removed joint Falsearm_el1
- removed joint Falsearm_f1x
- removed joint Falsearm_hr0
- removed joint Falsearm_sh0
- removed joint Falsearm_sh1
- removed joint Falsearm_wr0
- removed joint Falsearm_wr1
- removed joint Falsebase_link_joint
- removed joint Falsefront_left_foot
- removed joint Falsefront_left_hip_x
- removed joint Falsefront_left_hip_y
- removed joint Falsefront_left_knee
- removed joint Falsefront_rail_joint
- removed joint Falsefront_right_foot
- removed joint Falsefront_right_hip_x
- removed joint Falsefront_right_hip_y
- removed joint Falsefront_right_knee
- removed joint Falserear_left_foot
- removed joint Falserear_left_hip_x
- removed joint Falserear_left_hip_y
- removed joint Falserear_left_knee
- removed joint Falserear_rail_joint
- removed joint Falserear_right_foot
- removed joint Falserear_right_hip_x
- removed joint Falserear_right_hip_y
- removed joint Falserear_right_knee
- added joint arm_el0: type revolute, parent arm_link_hr0, child arm_link_el0, origin xyz=0.3385 0 0 rpy=0 0 0, axis 0 1 0, limit lower=0 upper=3.14159265358979311599 effort=90.9 velocity=10.0
- added joint arm_el1: type revolute, parent arm_link_el0, child arm_link_el1, origin xyz=0.40330 0.0 0.0750 rpy=0 0 0, axis 1 0 0, limit lower=-2.79252680319092716487 upper=2.79252680319092716487 effort=30.3 velocity=10.0
- added joint arm_f1x: type revolute, parent arm_link_wr1, child arm_link_fngr, origin xyz=0.11745 0 0.014820 rpy=0 0 0, axis 0.0 1.0 0.0, limit lower=-1.57 upper=0.0 effort=15.32 velocity=10.0
- added joint arm_hr0: type fixed, parent arm_link_sh1, child arm_link_hr0, origin xyz=0.0 0.0 0.0 rpy=0 0 0
- added joint arm_sh0: type revolute, parent body, child arm_link_sh0, origin xyz=0.292 0.0 0.188 rpy=0 0 0, axis 0 0 1, limit lower=-2.61799387799149441136 upper=3.14159265358979311599 effort=90.9 velocity=10.0
- added joint arm_sh1: type revolute, parent arm_link_sh0, child arm_link_sh1, origin xyz=0.0 0.0 0.0 rpy=0 0 0, axis 0 1 0, limit lower=-3.14159265358979311599 upper=0.52359877559829881565 effort=181.8 velocity=10.0
- added joint arm_wr0: type revolute, parent arm_link_el1, child arm_link_wr0, origin xyz=0.0 0.0 0.0 rpy=0 0 0, axis 0 1 0, limit lower=-1.83259571459404613236 upper=1.83259571459404613236 effort=30.3 velocity=10.0
- added joint arm_wr1: type revolute, parent arm_link_wr0, child arm_link_wr1, origin xyz=0.0 0.0 0.0 rpy=0 0 0, axis 1 0 0, limit lower=-2.87979326579064354163 upper=2.87979326579064354163 effort=30.3 velocity=10.0
- added joint base_link_joint: type fixed, parent body, child base_link, origin xyz=0 0 0 rpy=0 0 0
- added joint front_left_foot: type fixed, parent front_left_lower_leg, child front_left_ee, origin xyz=0 0 -0.35 rpy=0 0 0
- added joint front_left_hip_x: type revolute, parent body, child front_left_hip, origin xyz=0.29785 0.055 0 rpy=0 0 0, axis 1 0 0, limit lower=-0.78539816339744827899 upper=0.78539816339744827899 effort=45 velocity=17.647
- added joint front_left_hip_y: type revolute, parent front_left_hip, child front_left_upper_leg, origin xyz=0 0.110945 0 rpy=0 0 0, axis 0 1 0, limit lower=-0.89884456477707963539 upper=2.2951079663725435509 effort=45 velocity=17.647
- added joint front_left_knee: type revolute, parent front_left_upper_leg, child front_left_lower_leg, origin xyz=0.025 0 -0.3205 rpy=0 0 0, axis 0 1 0, limit lower=-2.7929 upper=-0.254801 effort=115 velocity=12.0
- added joint front_rail_joint: type fixed, parent body, child front_rail, origin xyz=0.223 0 0.0805 rpy=0 0 0
- added joint front_right_foot: type fixed, parent front_right_lower_leg, child front_right_ee, origin xyz=0 0 -0.35 rpy=0 0 0
- added joint front_right_hip_x: type revolute, parent body, child front_right_hip, origin xyz=0.29785 -0.055 0 rpy=0 0 0, axis 1 0 0, limit lower=-0.78539816339744827899 upper=0.78539816339744827899 effort=45 velocity=17.647
- added joint front_right_hip_y: type revolute, parent front_right_hip, child front_right_upper_leg, origin xyz=0 -0.110945 0 rpy=0 0 0, axis 0 1 0, limit lower=-0.89884456477707963539 upper=2.2951079663725435509 effort=45 velocity=17.647
- added joint front_right_knee: type revolute, parent front_right_upper_leg, child front_right_lower_leg, origin xyz=0.025 0 -0.3205 rpy=0 0 0, axis 0 1 0, limit lower=-2.7929 upper=-0.254801 effort=115 velocity=12.0
- added joint rear_left_foot: type fixed, parent rear_left_lower_leg, child rear_left_ee, origin xyz=0 0 -0.35 rpy=0 0 0
- added joint rear_left_hip_x: type revolute, parent body, child rear_left_hip, origin xyz=-0.29785 0.055 0 rpy=0 0 0, axis 1 0 0, limit lower=-0.78539816339744827899 upper=0.78539816339744827899 effort=45 velocity=17.647
- added joint rear_left_hip_y: type revolute, parent rear_left_hip, child rear_left_upper_leg, origin xyz=0 0.110945 0 rpy=0 0 0, axis 0 1 0, limit lower=-0.89884456477707963539 upper=2.2951079663725435509 effort=45 velocity=17.647
- added joint rear_left_knee: type revolute, parent rear_left_upper_leg, child rear_left_lower_leg, origin xyz=0.025 0 -0.3205 rpy=0 0 0, axis 0 1 0, limit lower=-2.7929 upper=-0.254801 effort=115 velocity=12.0
- added joint rear_rail_joint: type fixed, parent body, child rear_rail, origin xyz=-0.223 0 0.0805 rpy=0 0 0
- added joint rear_right_foot: type fixed, parent rear_right_lower_leg, child rear_right_ee, origin xyz=0 0 -0.35 rpy=0 0 0
- added joint rear_right_hip_x: type revolute, parent body, child rear_right_hip, origin xyz=-0.29785 -0.055 0 rpy=0 0 0, axis 1 0 0, limit lower=-0.78539816339744827899 upper=0.78539816339744827899 effort=45 velocity=17.647
- added joint rear_right_hip_y: type revolute, parent rear_right_hip, child rear_right_upper_leg, origin xyz=0 -0.110945 0 rpy=0 0 0, axis 0 1 0, limit lower=-0.89884456477707963539 upper=2.2951079663725435509 effort=45 velocity=17.647
- added joint rear_right_knee: type revolute, parent rear_right_upper_leg, child rear_right_lower_leg, origin xyz=0.025 0 -0.3205 rpy=0 0 0, axis 0 1 0, limit lower=-2.7929 upper=-0.254801 effort=115 velocity=12.0

File: spot_description/urdf/spot_macro.xacro (robot description, xacro)
@@ -2,5 +2,5 @@
 <robot name="spot" xmlns:xacro="http://www.ros.org/wiki/xacro">
     <xacro:include filename="$(find spot_description)/urdf/constants.urdf.xacro" />
-    <xacro:macro name="load_spot" params="arm:=false gazebo:=false tf_prefix">
+    <xacro:macro name="load_spot" params="arm gazebo tf_prefix">
         <link name="${tf_prefix}body">
             <visual>
