Commit message: Remove blank lines from URDF

File: spot_description/urdf/spot_macro.xacro (robot description, xacro)
@@ -1,8 +1,5 @@
 <?xml version="1.0"?>
 <robot name="spot" xmlns:xacro="http://www.ros.org/wiki/xacro">
-    <xacro:macro name="load_spot" params="
-    arm:=false
-    feet:=false
-    tf_prefix">
+    <xacro:macro name="load_spot" params="arm:=false feet:=false tf_prefix">
         <link name="${tf_prefix}body">
             <visual>

Commit message: Add missing collision geometries to Spot's URDF

File: spot_description/urdf/spot_macro.xacro (robot description, xacro)
@@ -60,4 +60,10 @@
                 </geometry>
             </visual>
+            <collision>
+                <geometry>
+                    <mesh
+                        filename="package://spot_description/meshes/base/visual/front_left_hip.obj" />
+                </geometry>
+            </collision>
             <inertial>
                 <origin rpy="-0.716521349312305 0.02956473059648479 0.03655230014702582"
@@ -146,4 +152,10 @@
                 </geometry>
             </visual>
+            <collision>
+                <geometry>
+                    <mesh
+                        filename="package://spot_description/meshes/base/visual/front_right_hip.obj" />
+                </geometry>
+            </collision>
             <inertial>
                 <origin rpy="0.7165213493123055 -0.02956473059648479 0.03655230014702582"
@@ -232,4 +244,10 @@
                 </geometry>
             </visual>
+            <collision>
+                <geometry>
+                    <mesh
+                        filename="package://spot_description/meshes/base/visual/rear_left_hip.obj" />
+                </geometry>
+            </collision>
             <inertial>
                 <origin rpy="0.7165213493123055 -0.02956473059648479 0.03655230014702582"
@@ -318,4 +336,10 @@
                 </geometry>
             </visual>
+            <collision>
+                <geometry>
+                    <mesh
+                        filename="package://spot_description/meshes/base/visual/rear_right_hip.obj" />
+                </geometry>
+            </collision>
             <inertial>
                 <origin rpy="0.7165213493123055 -0.02956473059648479 0.03655230014702582"
